File: kiCad/pterodactyl.kicad_pcb (KiCad board)
At the start: 2 copper layers, 327.7 x 165.9 mm, 153 parts, among them J0 Conn_01x03, SW0 MX, SW1 MX, SW10 MX, SW11 MX, SW12 MX, SW13 MX, SW14 MX, SW15 MX, SW16 MX, SW17 MX, SW18 MX, SW19 MX, SW2 MX, SW20 MX, SW21 MX, SW22 MX, SW23 MX, SW24 MX, SW25 MX, SW26 MX, SW27 MX, SW28 MX, SW29 MX, SW3 MX, SW30 MX, SW31 MX, SW32 MX, SW33 MX, SW34 MX, SW35 MX, SW36 MX, SW37 MX, SW38 MX, SW39 MX, SW4 MX, SW40 MX, SW41 MX, SW42 MX, SW43 MX, SW44 MX, SW45 MX, SW46 MX, SW47 MX, SW48 MX, SW49 MX, SW5 MX, SW50 MX, SW51 MX, SW52 MX, SW53 MX, SW54 MX, SW55 MX, SW56 MX, SW57 MX, SW58 MX, SW59 MX, SW6 MX, SW60 MX, SW61 RotaryEncoder_Switch, SW62 MX, SW63 MX, SW64 MX, SW65 MX, SW66 MX, SW67 MX, SW68 MX, SW69 MX, SW7 MX, SW70 MX, SW71 MX, SW8 MX, SW9 MX, U0 Sparkfun_Pro_Micro

Commit message: finish routing
Parts:
- moved SW71 98.3 mm to (201.3, 95.8)
- moved J0 54.8 mm to (203.8, 90.6), turned to -90 degrees
- renumbered D60 to D12, D61 to D13, D62 to D14, D12 to D15, D13 to D16, D14 to D17, D15 to D18, D16 to D19, D17 to D20, D18 to D21, D19 to D22, D20 to D23, D21 to D24, D22 to D25, D23 to D26, D63 to D27, D64 to D28, D65 to D29, D70 to D30, D24 to D31, D25 to D32, D26 to D33, D27 to D34, D28 to D35, D29 to D36, D30 to D37, D31 to D38, D32 to D39, D33 to D40, D34 to D41, D35 to D42, D66 to D43, D67 to D44, D68 to D45, D69 to D46, D36 to D47, D37 to D48, D38 to D49, D39 to D50, D40 to D51, D41 to D52, D42 to D53, D43 to D54, D44 to D55, D45 to D56, D46 to D57, D47 to D58, D48 to D59, D49 to D60, D50 to D61, D51 to D62, D52 to D63, D53 to D64, D54 to D65, D55 to D66, D56 to D67, D57 to D68, D58 to D69, D59 to D70, SW1 to SW0, SW2 to SW1, SW11 to SW10, SW12 to SW11, SW62 to SW12, SW63 to SW13, SW64 to SW14, SW61 to SW15, SW13 to SW16, SW14 to SW17, SW15 to SW18, SW16 to SW19, SW3 to SW2, SW17 to SW20, SW18 to SW21, SW19 to SW22, SW20 to SW23, SW21 to SW24, SW22 to SW25, SW23 to SW26, SW24 to SW27, SW65 to SW28, SW66 to SW29, SW4 to SW3, SW67 to SW30, SW25 to SW31, SW26 to SW32, SW27 to SW33, SW28 to SW34, SW29 to SW35, SW30 to SW36, SW31 to SW37, SW32 to SW38, SW33 to SW39, SW5 to SW4, SW34 to SW40, SW35 to SW41, SW36 to SW42, SW68 to SW43, SW69 to SW44, SW70 to SW45, SW71 to SW46, SW37 to SW47, SW38 to SW48, SW39 to SW49, SW6 to SW5, SW40 to SW50, SW41 to SW51, SW42 to SW52, SW43 to SW53, SW44 to SW54, SW45 to SW55, SW46 to SW56, SW47 to SW57, SW48 to SW58, SW49 to SW59, SW7 to SW6, SW50 to SW60, SW51 to SW61, SW52 to SW62, SW53 to SW63, SW54 to SW64, SW55 to SW65, SW56 to SW66, SW57 to SW67, SW58 to SW68, SW59 to SW69, SW8 to SW7, SW60 to SW70, SW0 to SW71, SW9 to SW8, SW10 to SW9
Connections:
- D31 pad 1: /COL8 -> /ROW2
- D32 pad 1: /COL8 -> /ROW2
- D33 pad 1: /COL8 -> /ROW2
- D34 pad 1: /COL8 -> /ROW2
- D35 pad 1: /COL8 -> /ROW2
- D36 pad 1: /COL8 -> /ROW2
- D37 pad 1: /COL8 -> /ROW2
- D38 pad 1: /COL8 -> /ROW2
- D39 pad 1: /COL8 -> /ROW2
- D40 pad 1: /COL8 -> /ROW2
- D41 pad 1: /COL8 -> /ROW2
- D42 pad 1: /COL8 -> /ROW2
- D42 pad 2: /COL8 -> /ROW2
- D43 pad 1: /COL8 -> /ROW2
- D44 pad 1: /COL8 -> /ROW2
- D45 pad 1: /COL8 -> /ROW2
- D46 pad 1: /COL8 -> /ROW2
- SW13 pad 1: /COL7 -> /COL6
- SW14 pad 1: /COL8 -> /COL7
- SW15 pad S2: /COL8 -> /COL7
- SW29 pad 1: /COL7 -> /COL6
- SW30 pad 1: /COL8 -> /COL7
- SW42 pad 2: /COL8 -> /ROW2
- SW44 pad 1: /COL7 -> /COL6
- SW45 pad 1: /COL8 -> /COL7
- SW46 pad 1: /COL8 -> /COL7
- U0 pad 1: /ROTA -> unconnected-(U0-D1/TX-Pad1)
- U0 pad 11: /COL3 -> /COL5
- U0 pad 12: /COL2 -> /ROW0
- U0 pad 13: /ROW4 -> /ROW2
- U0 pad 14: /ROW3 -> /ROW4
- U0 pad 15: /COL8 -> /ROW3
- U0 pad 18: /ROW0 -> /COL2
- U0 pad 5: unconnected-(U0-D2-Pad5) -> /ROTA
- U0 pad 6: /COL8 -> unconnected-(U0-~D3-Pad6)
- U0 pad 9: /COL5 -> /COL3
Routing:
- net /ROW2: track 0.00 -> 363.4 mm
- net /COL8: track 277.0 -> 0.00 mm
- net /ROW4: track 181.1 -> 424.4 mm
- net /ROW3: track 172.4 -> 378.7 mm, vias 0 -> 1
- net GND: track 0.00 -> 168.8 mm
- net /ROTB: track 0.00 -> 133.8 mm
- net /ROTA: track 0.00 -> 123.5 mm
- net /COL5: track 152.4 -> 268.4 mm, vias 0 -> 1
- net /COL6: track 35.6 -> 143.9 mm
- net /ROW1: track 195.3 -> 298.0 mm
- net /ROW0: track 178.0 -> 274.2 mm, vias 0 -> 1
- net /COL0: track 174.2 -> 265.2 mm
- net /COL7: track 35.6 -> 118.9 mm
- net /COL4: track 152.4 -> 229.7 mm, vias 0 -> 1
- net /COL1: track 173.0 -> 226.1 mm
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
Commit message: add edge cuts, flip controller
Parts:
- J0, SW71: moved to B.Cu
- U0: moved to F.Cu
- moved J0 1.96 mm to (203.8, 88.6), turned to 90 degrees
- turned SW71 to 180 degrees
Connections:
- U0 pad 10: /COL4 -> /ROW3
- U0 pad 11: /COL5 -> /ROW4
- U0 pad 12: /ROW0 -> /ROW2
- U0 pad 13: /ROW2 -> /ROW0
- U0 pad 14: /ROW4 -> /COL5
- U0 pad 15: /ROW3 -> /COL4
- U0 pad 16: /ROW1 -> /COL3
- U0 pad 17: /PIN15 -> /COL6
- U0 pad 18: /COL2 -> /COL7
- U0 pad 19: /COL1 -> /ROTA
- U0 pad 2: /ROTB -> unconnected-(U0-D0/RX-Pad2)
- U0 pad 20: /COL0 -> /ROTB
- U0 pad 5: /ROTA -> /COL0
- U0 pad 6: unconnected-(U0-~D3-Pad6) -> /COL1
- U0 pad 7: /COL7 -> /COL2
- U0 pad 8: /COL6 -> /PIN15
- U0 pad 9: /COL3 -> /ROW1
Routing:
- net /ROTB: track 133.8 -> 126.2 mm
- net +5V: track 5.10 -> 12.1 mm
- net GND: track 168.8 -> 162.6 mm, vias 0 -> 1
- net /PIN15: track 14.8 -> 18.8 mm
- net /ROTA: track 123.5 -> 121.0 mm
- net Net-(D14-A): vias 2 -> 1
- net Net-(D13-A): vias 2 -> 1
Other:
- board size 327.7 x 165.9 mm -> 324.8 x 157.5 mm

Commit message: rewire everything, change ergonomics
Parts:
- removed ? (x8): , 
- removed U0: Sparkfun_Pro_Micro, Keebio-Parts:ArduinoProMicro
- added G***: LOGO, keyswitches:batman, F.Cu at (185.2, 393.2)
- added U1: Elite-C, Keebio-Parts:Elite-C, F.Cu at (210.7, 85.3)
- moved J0 132.5 mm to (231.1, 218.3)
- moved SW71 132.5 mm to (228.6, 225.4)
- moved SW11 54.1 mm to (375.2, 67.8), turned to 17 degrees
- moved D10 53.6 mm to (366.6, 72.9), turned to 107 degrees
- moved SW10 53.5 mm to (356.9, 73.3), turned to 17 degrees
- moved D11 53.2 mm to (374.3, 78.0), turned to 17 degrees
- moved D9 53.0 mm to (348.5, 78.4), turned to 107 degrees
- moved SW9 52.9 mm to (338.7, 78.9), turned to 17 degrees
- moved SW27 52.6 mm to (380.7, 86.0), turned to 17 degrees
- moved D8 52.4 mm to (330.3, 84.0), turned to 107 degrees
- moved SW8 52.4 mm to (320.5, 84.5), turned to 17 degrees
- moved D25 52.0 mm to (372.3, 91.1), turned to 107 degrees
- moved D7 51.9 mm to (312.1, 89.6), turned to 107 degrees
- moved SW26 51.9 mm to (362.5, 91.6), turned to 17 degrees
- moved SW7 51.9 mm to (302.3, 90.1), turned to 17 degrees
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Connections:
- D0 pad 1: /ROW0 -> /ROW1
- D10 pad 1: /ROW0 -> /ROW1
- D12 pad 1: /ROW0 -> /ROW1
- D14 pad 1: /ROW0 -> /ROW1
- D15 pad 1: /ROW1 -> /ROW3
- D16 pad 1: /ROW1 -> /ROW2
- D17 pad 1: /ROW1 -> /ROW3
- D18 pad 1: /ROW1 -> /ROW2
- D19 pad 1: /ROW1 -> /ROW3
- D2 pad 1: /ROW0 -> /ROW1
- D20 pad 1: /ROW1 -> /ROW2
- D21 pad 1: /ROW1 -> /ROW3
- D22 pad 1: /ROW1 -> /ROW2
- D23 pad 1: /ROW1 -> /ROW3
- D24 pad 1: /ROW1 -> /ROW2
- D25 pad 1: /ROW1 -> /ROW3
- D26 pad 1: /ROW1 -> /ROW2
- D27 pad 1: /ROW1 -> /ROW3
- D28 pad 1: /ROW1 -> /ROW2
- D29 pad 1: /ROW1 -> /ROW3
- D30 pad 1: /ROW1 -> /ROW2
- D31 pad 1: /ROW2 -> /ROW5
- D32 pad 1: /ROW2 -> /ROW4
- D33 pad 1: /ROW2 -> /ROW5
- D34 pad 1: /ROW2 -> /ROW4
- D35 pad 1: /ROW2 -> /ROW5
- D36 pad 1: /ROW2 -> /ROW4
- D37 pad 1: /ROW2 -> /ROW5
- D38 pad 1: /ROW2 -> /ROW4
- D39 pad 1: /ROW2 -> /ROW5
- D4 pad 1: /ROW0 -> /ROW1
- D40 pad 1: /ROW2 -> /ROW4
- D41 pad 1: /ROW2 -> /ROW5
- D42 pad 1: /ROW2 -> /ROW4
- D42 pad 2: /ROW2 -> Net-(D42-A)
- D43 pad 1: /ROW2 -> /ROW5
- D44 pad 1: /ROW2 -> /ROW4
- D45 pad 1: /ROW2 -> /ROW5
- D46 pad 1: /ROW2 -> /ROW4
- D47 pad 1: /ROW3 -> /ROW7
- D48 pad 1: /ROW3 -> /ROW6
- D49 pad 1: /ROW3 -> /ROW7
- D50 pad 1: /ROW3 -> /ROW6
- D51 pad 1: /ROW3 -> /ROW7
- D52 pad 1: /ROW3 -> /ROW6
- D53 pad 1: /ROW3 -> /ROW7
- D54 pad 1: /ROW3 -> /ROW6
- D55 pad 1: /ROW3 -> /ROW7
- D56 pad 1: /ROW3 -> /ROW6
- D57 pad 1: /ROW3 -> /ROW7
- D58 pad 1: /ROW3 -> /ROW6
- D59 pad 1: /ROW4 -> /ROW9
- D6 pad 1: /ROW0 -> /ROW1
- D60 pad 1: /ROW4 -> /ROW8
- D61 pad 1: /ROW4 -> /ROW9
- D62 pad 1: /ROW4 -> /ROW8
- D63 pad 1: /ROW4 -> /ROW9
- D64 pad 1: /ROW4 -> /ROW8
- D65 pad 1: /ROW4 -> /ROW9
- D66 pad 1: /ROW4 -> /ROW8
- D67 pad 1: /ROW4 -> /ROW9
- D68 pad 1: /ROW4 -> /ROW8
- D69 pad 1: /ROW4 -> /ROW9
- D70 pad 1: /ROW4 -> /ROW8
- D8 pad 1: /ROW0 -> /ROW1
- SW42 pad 2: /ROW2 -> Net-(D42-A)
Routing:
- net /ROW4: track 424.4 -> 0.00 mm
- net /ROW3: track 378.7 -> 0.00 mm, vias 1 -> 0
- net /ROW2: track 363.4 -> 0.00 mm
- net /ROW1: track 298.0 -> 0.00 mm
- net /ROW0: track 274.2 -> 0.00 mm, vias 1 -> 0
- net /COL5: track 268.4 -> 0.00 mm, vias 1 -> 0
- net /COL0: track 265.2 -> 0.00 mm
- net /COL4: track 229.7 -> 0.00 mm, vias 1 -> 0
- net /COL1: track 226.1 -> 0.00 mm
- net /COL3: track 191.3 -> 0.00 mm, vias 1 -> 0
- net /COL2: track 188.0 -> 0.00 mm
- net GND: track 162.6 -> 0.00 mm, vias 1 -> 0
- net /COL6: track 143.9 -> 0.00 mm
- net /ROTB: track 126.2 -> 0.00 mm
- net /ROTA: track 121.0 -> 0.00 mm
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Other:
- board outline removed
- board text added: "The angle of each side is 17 degrees. Bottom distance is 18cm. Top distance is 12.5cm"

Commit message: fix annotations, start routing
Parts:
- removed U1: Elite-C, Keebio-Parts:Elite-C
- added D71: 1N4148, Diode_THT:D_DO-35_SOD27_P7.62mm_Horizontal, F.Cu at (315.0, 204.0)
- added D72: 1N4148, Diode_THT:D_DO-35_SOD27_P7.62mm_Horizontal, F.Cu at (333.3, 198.5)
- added D73: 1N4148, Diode_THT:D_DO-35_SOD27_P7.62mm_Horizontal, F.Cu at (351.5, 192.9)
- added D74: 1N4148, Diode_THT:D_DO-35_SOD27_P7.62mm_Horizontal, F.Cu at (369.8, 187.3)
- added D75: 1N4148, Diode_THT:D_DO-35_SOD27_P7.62mm_Horizontal, F.Cu at (388.0, 181.7)
- added SW72: MX, keyswitches:Kailh_socket_MX, F.Cu at (341.9, 191.8)
- added SW73: MX, keyswitches:Kailh_socket_MX, F.Cu at (360.2, 186.3)
- added SW74: MX, keyswitches:Kailh_socket_MX, F.Cu at (378.4, 180.7)
- added SW75: MX, keyswitches:Kailh_socket_MX, F.Cu at (396.6, 175.1)
- added SW76: MX, Molex-0548190589:PushButton_6x6mm_TH_Pretty, F.Cu at (182.2, 198.3)
- added U0: Elite-C, Keebio-Parts:Elite-C, F.Cu at (210.6, 120.3)
- J0: moved to F.Cu
- SW15: value RotaryEncoder_Switch -> MX; footprint Keebio-Parts:RotaryEncoder_EC11 -> keyswitches:Kailh_socket_MX
- SW6: value MX -> RotaryEncoder_Switch; footprint keyswitches:Kailh_socket_MX -> Keebio-Parts:RotaryEncoder_EC11
- SW71: footprint Molex-0548190589:PushButton_6x6mm_TH_Pretty -> keyswitches:Kailh_socket_MX; moved to F.Cu
- moved SW47 354.7 mm to (385.5, 138.8), turned to 17 degrees
- moved SW31 343.6 mm to (380.0, 120.7), turned to 17 degrees
- moved D47 337.8 mm to (376.9, 145.4), turned to 107 degrees
- moved D31 334.3 mm to (371.4, 127.3), turned to 107 degrees
- moved D60 331.0 mm to (364.2, 169.2), turned to 107 degrees
- moved D61 330.4 mm to (382.5, 163.6), turned to 107 degrees
- moved SW59 330.2 mm to (354.6, 168.1), turned to 17 degrees
- moved SW60 329.5 mm to (372.9, 162.5), turned to 17 degrees
- moved SW61 329.1 mm to (391.1, 157.0), turned to 17 degrees
- moved D15 323.2 mm to (365.8, 109.2), turned to 107 degrees
- moved D59 317.0 mm to (346.0, 174.7), turned to 107 degrees
- moved D68 254.6 mm to (122.9, 209.3), turned to 73 degrees
- moved D67 252.2 mm to (104.8, 203.7), turned to 73 degrees
- moved D66 250.4 mm to (86.5, 198.1), turned to 73 degrees
- moved D65 249.1 mm to (68.2, 192.5), turned to 73 degrees
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Connections:
- D15 pad 1: /ROW3 -> /ROW0
- D16 pad 1: /ROW2 -> /ROW3
- D17 pad 1: /ROW3 -> /ROW2
- D18 pad 1: /ROW2 -> /ROW3
- D19 pad 1: /ROW3 -> /ROW2
- D20 pad 1: /ROW2 -> /ROW3
- D21 pad 1: /ROW3 -> /ROW2
- D22 pad 1: /ROW2 -> /ROW3
- D23 pad 1: /ROW3 -> /ROW2
- D24 pad 1: /ROW2 -> /ROW3
- D25 pad 1: /ROW3 -> /ROW2
- D26 pad 1: /ROW2 -> /ROW3
- D27 pad 1: /ROW3 -> /ROW2
- D28 pad 1: /ROW2 -> /ROW3
- D29 pad 1: /ROW3 -> /ROW2
- D30 pad 1: /ROW2 -> /ROW3
- D31 pad 1: /ROW5 -> /ROW2
- D32 pad 1: /ROW4 -> /ROW5
- D33 pad 1: /ROW5 -> /ROW4
- D34 pad 1: /ROW4 -> /ROW5
- D35 pad 1: /ROW5 -> /ROW4
- D36 pad 1: /ROW4 -> /ROW5
- D37 pad 1: /ROW5 -> /ROW4
- D38 pad 1: /ROW4 -> /ROW5
- D39 pad 1: /ROW5 -> /ROW4
- D40 pad 1: /ROW4 -> /ROW5
- D41 pad 1: /ROW5 -> /ROW4
- D42 pad 1: /ROW4 -> /ROW5
- D43 pad 1: /ROW5 -> /ROW4
- D44 pad 1: /ROW4 -> /ROW5
- D45 pad 1: /ROW5 -> /ROW4
- D46 pad 1: /ROW4 -> /ROW5
- D47 pad 1: /ROW7 -> /ROW4
- D48 pad 1: /ROW6 -> /ROW7
- D49 pad 1: /ROW7 -> /ROW6
- D50 pad 1: /ROW6 -> /ROW7
- D51 pad 1: /ROW7 -> /ROW6
- D52 pad 1: /ROW6 -> /ROW7
- D53 pad 1: /ROW7 -> /ROW6
- D54 pad 1: /ROW6 -> /ROW7
- D55 pad 1: /ROW7 -> /ROW6
- D56 pad 1: /ROW6 -> /ROW7
- D57 pad 1: /ROW7 -> /ROW6
- D58 pad 1: /ROW6 -> /ROW7
- D59 pad 1: /ROW9 -> /ROW6
- D60 pad 1: /ROW8 -> /ROW7
- D61 pad 1: /ROW9 -> /ROW6
- D62 pad 1: /ROW8 -> /ROW9
- D63 pad 1: /ROW9 -> /ROW8
- D64 pad 1: /ROW8 -> /ROW9
- D65 pad 1: /ROW9 -> /ROW8
- D66 pad 1: /ROW8 -> /ROW9
- D67 pad 1: /ROW9 -> /ROW8
- D68 pad 1: /ROW8 -> /ROW9
- D69 pad 1: /ROW9 -> /ROW8
- D70 pad 1: /ROW8 -> /ROW9
- SW16 pad 2: Net-(D15-A) -> Net-(D16-A)
- SW17 pad 2: Net-(D16-A) -> Net-(D17-A)
- SW18 pad 2: Net-(D17-A) -> Net-(D18-A)
- SW19 pad 2: Net-(D18-A) -> Net-(D19-A)
- SW20 pad 2: Net-(D19-A) -> Net-(D20-A)
- SW21 pad 2: Net-(D20-A) -> Net-(D21-A)
- SW22 pad 2: Net-(D21-A) -> Net-(D22-A)
- SW23 pad 2: Net-(D22-A) -> Net-(D23-A)
- SW24 pad 2: Net-(D23-A) -> Net-(D24-A)
- SW25 pad 2: Net-(D24-A) -> Net-(D25-A)
- SW26 pad 2: Net-(D25-A) -> Net-(D26-A)
- SW27 pad 2: Net-(D26-A) -> Net-(D27-A)
- SW28 pad 2: Net-(D27-A) -> Net-(D28-A)
- SW29 pad 2: Net-(D28-A) -> Net-(D29-A)
- SW30 pad 2: Net-(D29-A) -> Net-(D30-A)
- SW31 pad 1: /COL0 -> /COL7
- SW33 pad 1: /COL1 -> /COL0
- SW35 pad 1: /COL2 -> /COL1
- SW37 pad 1: /COL3 -> /COL2
- SW39 pad 1: /COL4 -> /COL3
- SW41 pad 1: /COL5 -> /COL4
- SW43 pad 1: /COL6 -> /COL5
- SW45 pad 1: /COL7 -> /COL6
- SW47 pad 1: /COL0 -> /COL7
- SW49 pad 1: /COL1 -> /COL0
- SW51 pad 1: /COL2 -> /COL1
- SW53 pad 1: /COL3 -> /COL2
- SW56 pad 1: /COL4 -> /COL5
- SW58 pad 1: /COL5 -> /COL6
- SW59 pad 1: /COL0 -> /COL6
- SW60 pad 1: /COL0 -> /COL7
- SW61 pad 1: /COL1 -> /COL7
- SW62 pad 1: /COL1 -> /COL0
- SW63 pad 1: /COL2 -> /COL0
- SW64 pad 1: /COL2 -> /COL1
- SW65 pad 1: /COL3 -> /COL1
- SW66 pad 1: /COL3 -> /COL2
- SW67 pad 1: /COL4 -> /COL2
- SW68 pad 1: /COL4 -> /COL3
- SW69 pad 1: /COL5 -> /COL4
- SW71 pad 1: Net-(U1-RST) -> /COL5
- SW71 pad 2: GND -> Net-(D71-A)
Routing:
- net Net-(D0-A): track 0.00 -> 12.6 mm
- net Net-(D16-A): track 0.00 -> 12.6 mm
- net Net-(D32-A): track 0.00 -> 12.1 mm
- net Net-(D48-A): track 0.00 -> 12.0 mm
- net Net-(D30-A): track 0.00 -> 3.12 mm
- net Net-(D74-A): track 0.00 -> 3.12 mm
- net Net-(D46-A): track 0.00 -> 3.12 mm
- net Net-(D60-A): track 0.00 -> 3.12 mm
- net Net-(D73-A): track 0.00 -> 3.11 mm
- net Net-(D45-A): track 0.00 -> 3.11 mm
- net Net-(D59-A): track 0.00 -> 3.11 mm
- net Net-(D29-A): track 0.00 -> 3.11 mm
- net Net-(D44-A): track 0.00 -> 3.09 mm
- net Net-(D58-A): track 0.00 -> 3.09 mm
- net Net-(D28-A): track 0.00 -> 3.09 mm
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Other:
- board text removed: "The angle of each side is 17 degrees. Bottom distance is 18cm. Top distance is 12.5cm"

Commit message: add most of routing
Parts:
- moved SW76 105.5 mm to (254.6, 121.6)
- moved J0 82.6 mm to (260.9, 120.4)
- moved D41 46.5 mm to (229.9, 139.1)
- moved D40 46.2 mm to (234.3, 139.1)
- moved D6 28.7 mm to (207.6, 139.1)
- moved D7 28.4 mm to (203.1, 139.1)
- moved D22 18.6 mm to (198.6, 139.1)
- moved D25 18.6 mm to (221.0, 139.1)
- moved D23 18.3 mm to (194.2, 139.1)
- moved D24 18.3 mm to (225.4, 139.1)
- moved D8 10.6 mm to (216.5, 139.1)
- moved D9 10.3 mm to (212.0, 139.1)
- moved D38 8.78 mm to (189.7, 139.1)
- moved D39 8.48 mm to (185.2, 139.1)
- moved U0 7.73 mm to (209.8, 112.6)
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Connections:
- U0 pad 10: /ROW4 -> /ROW5
- U0 pad 11: /ROW5 -> /ROW7
- U0 pad 12: /ROW6 -> /ROW9
- U0 pad 13: /COL7 -> /ROW8
- U0 pad 14: /COL6 -> /ROW6
- U0 pad 15: /COL5 -> /ROW4
- U0 pad 16: /COL4 -> /ROW2
- U0 pad 17: /COL3 -> /ROW0
- U0 pad 18: /ROW9 -> /COL5
- U0 pad 19: /ROW8 -> /COL6
- U0 pad 20: /ROW7 -> /COL7
- U0 pad 6: /ROW0 -> /COL3
- U0 pad 7: /ROW1 -> /COL4
- U0 pad 8: /ROW2 -> /ROW1
Routing:
- net /ROW6: track 0.00 -> 535.9 mm
- net /ROW7: track 0.00 -> 527.7 mm, vias 0 -> 1
- net /ROW8: track 0.00 -> 504.6 mm
- net /ROW9: track 0.00 -> 504.5 mm, vias 0 -> 1
- net /ROW5: track 0.00 -> 487.5 mm
- net /ROW4: track 0.00 -> 466.1 mm
- net /ROW3: track 0.00 -> 459.8 mm
- net /ROW2: track 0.00 -> 420.6 mm
- net /ROW0: track 0.00 -> 392.3 mm
- net /ROW1: track 0.00 -> 376.3 mm
- net /COL7: track 0.00 -> 261.3 mm
- net /COL4: track 0.00 -> 250.5 mm
- net /COL0: track 0.00 -> 247.8 mm
- net /COL3: track 0.00 -> 226.8 mm
- net /COL6: track 0.00 -> 224.0 mm
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Other:
- board outline added: 399.4 x 138 mm

Commit message: finish routing, add edge cuts, add artwork
Parts:
- removed the G*** at (199.4, 443.9)
- added G***: LOGO, pterodactyl:pteranodon, F.Cu at (209.7, 155.9)
- added G***: LOGO, pterodactyl:pteranodon_big, B.Cu at (196.7, 163.1)
- J0, SW76: moved to B.Cu
- moved J0 51.6 mm to (209.8, 113.6)
- moved SW76 48.0 mm to (209.8, 104.5), turned to 90 degrees
Routing:
- net /ROTB: track 0.00 -> 101.4 mm
- net GND: track 18.8 -> 118.0 mm
- net /ROTA: track 0.00 -> 89.2 mm
- net /COL0: track 247.8 -> 320.7 mm
- net /COL1: track 209.6 -> 280.3 mm
- net /COL2: track 172.5 -> 238.8 mm, vias 0 -> 1
- net /COL7: track 261.3 -> 326.6 mm, vias 0 -> 1
- net /COL6: track 224.0 -> 287.8 mm
- net /COL5: track 186.4 -> 249.5 mm
- net Net-(D38-A): track 97.6 -> 124.3 mm
- net Net-(D39-A): track 116.3 -> 140.3 mm
- net Net-(D62-A): track 0.00 -> 18.4 mm
- net /PIN15: track 0.00 -> 13.0 mm
- net +5V: track 0.00 -> 9.25 mm
- net Net-(U0-RST): track 0.00 -> 6.42 mm
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Other:
- board size 399.4 x 138 mm -> 396.4 x 134.8 mm
- board text added: "Pterodactyl by SylivanKenobi"
