File: kiCad/pteranodon.kicad_pcb (KiCad board)
At the start: 2 copper layers, 396.4 x 134.8 mm, 157 parts, among them J0 Conn_01x03, SW0 MX, SW1 MX, SW10 MX, SW11 MX, SW12 MX, SW13 MX, SW14 MX, SW15 MX, SW16 MX, SW17 MX, SW18 MX, SW19 MX, SW2 MX, SW20 MX, SW21 MX, SW22 MX, SW23 MX, SW24 MX, SW25 MX, SW26 MX, SW27 MX, SW28 MX, SW29 MX, SW3 MX, SW30 MX, SW31 MX, SW32 MX, SW33 MX, SW34 MX, SW35 MX, SW36 MX, SW37 MX, SW38 MX, SW39 MX, SW4 MX, SW40 MX, SW41 MX, SW42 MX, SW43 MX, SW44 MX, SW45 MX, SW46 MX, SW47 MX, SW48 MX, SW49 MX, SW5 MX, SW50 MX, SW51 MX, SW52 MX, SW53 MX, SW54 MX, SW55 MX, SW56 MX, SW57 MX, SW58 MX, SW59 MX, SW6 RotaryEncoder_Switch, SW60 MX, SW61 MX, SW62 MX, SW63 MX, SW64 MX, SW65 MX, SW66 MX, SW67 MX, SW68 MX, SW69 MX, SW7 MX, SW70 MX, SW71 MX, SW72 MX, SW73 MX, SW74 MX, SW75 MX, SW76 MX, SW8 MX, SW9 MX, U0 Elite-C

Commit message: add mounting points, cleanup some footprints
Parts:
- removed the G*** at (209.7, 155.9)
- removed the G*** at (196.7, 163.1)
- added ?: , , F.Cu at (368.9, 108.1)
- added ?: , , F.Cu at (295.9, 130.4)
- added ?: , , F.Cu at (33.7, 162.5)
- added ?: , , F.Cu at (50.4, 108.1)
- added ?: , , F.Cu at (211.2, 179.9)
- added ?: , , F.Cu at (123.4, 130.4)
- added ?: , , F.Cu at (312.6, 184.8)
- added ?: , , F.Cu at (385.6, 162.5)
- added ?: , , F.Cu at (211.2, 198.9)
- added ?: , , F.Cu at (106.8, 184.8)
- added G***: LOGO, pteranodon:pteranodon, F.Cu at (209.4, 153.8)
- added G***: LOGO, pteranodon:pteranodon_big, B.Cu at (196.3, 160.9)
- D0, D1, D10, D11, D12, D13, D14, D15, D16, D17, D18, D19, D2, D20, D21, D22, D23, D24, D25, D26, D27, D28, D29, D3, D30, D31, D32, D33, D34, D35, D36, D37, D38, D39, D4, D40, D41, D42, D43, D44, D45, D46, D47, D48, D49, D5, D50, D51, D52, D53, D54, D55, D56, D57, D58, D59, D6, D60, D61, D62, D63, D64, D65, D66, D67, D68, D69, D7, D70, D71, D72, D73, D74, D75, D8, D9: footprint Diode_THT:D_DO-35_SOD27_P7.62mm_Horizontal -> pteranodon:D_DO-35_SOD27_P7.62mm_Horizontal
- moved SW67 2.11 mm to (113.2, 196.7)
- moved D55 2.11 mm to (288.2, 192.2)
- moved D27 2.11 mm to (299.2, 143.3)
- moved D44 2.11 mm to (323.0, 155.8)
- moved D57 2.11 mm to (310.3, 179.6)
- moved D60 2.11 mm to (365.0, 162.8)
- moved SW26 2.11 mm to (289.6, 142.2)
- moved SW55 2.11 mm to (282.4, 184.1)
- moved SW35 2.11 mm to (87.7, 149.2)
- moved SW37 2.11 mm to (124.3, 160.4)
- moved SW50 2.11 mm to (63.9, 161.8)
- moved SW63 2.11 mm to (40.1, 174.4)
- moved SW48 2.11 mm to (27.4, 150.6)
- moved D50 2.11 mm to (53.1, 162.5)
- moved D37 2.11 mm to (113.4, 161.1)
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Routing:
- net /ROW1: track 378.8 -> 377.7 mm
Other:
- outline, holes or cut-outs redrawn
- board text added: "Pteranodon by SylivanKenobi"
- board text removed: "Pterodactyl by SylivanKenobi"
